File: v2/HWDesign/EAGLE/bluz_proto_v2_revA.brd (EAGLE design)
At the start: 45.7 x 57.1 mm, 72 parts

Commit message: add more breakouts. add decoupling cap
Parts:
- added C1: (no value), SparkFun-Capacitors:0603-CAP
- added JP15, JP16: (no value), SparkFun-Connectors:1X08_NO_SILK
Connections:
- net GND: now also C1.2
- net VCC: now also C1.1
Routing:
- net VCC: track 47.0 -> 48.7 mm
Changed lines of the file:
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@@
 <attribute name="VALUE" x="40.259" y="31.242" size="0.4064" layer="27" rot="R180"/>
+</element>
+<element name="C1" library="SparkFun-Capacitors" package="0603-CAP" value="" x="6.35" y="35.56" rot="R180"/>
+<element name="JP15" library="SparkFun-Connectors" package="1X08_NO_SILK" value="" x="11.43" y="38.1" smashed="yes" rot="R90">
+<attribute name="VALUE" x="14.605" y="36.83" size="1.27" layer="27" rot="R90"/>
+</element>
+<element name="JP16" library="SparkFun-Connectors" package="1X08_NO_SILK" value="" x="34.29" y="38.1" smashed="yes" rot="R90">
+<attribute name="VALUE" x="37.465" y="36.83" size="1.27" layer="27" rot="R90"/>
 </element>
 </elements>
@@
 <wire x1="8.89" y1="50.8" x2="8.89" y2="53.34" width="0.4064" layer="1"/>
 <wire x1="31.75" y1="31.75" x2="31.75" y2="35.56" width="0.6096" layer="1"/>
-<wire x1="31.75" y1="35.56" x2="8.89" y2="35.56" width="0.6096" layer="1"/>
+<wire x1="31.75" y1="35.56" x2="10.16" y2="35.56" width="0.6096" layer="1"/>
+<wire x1="10.16" y1="35.56" x2="8.89" y2="35.56" width="0.6096" layer="1"/>
 <wire x1="8.89" y1="35.56" x2="8.89" y2="38.1" width="0.6096" layer="1"/>
+<contactref element="C1" pad="1"/>
+<wire x1="7.2" y1="35.56" x2="8.89" y2="35.56" width="0.6096" layer="1"/>
 </signal>
 <signal name="GND">
@@
 <via x="22.86" y="11.43" extent="1-16" drill="0.6"/>
 <via x="22.86" y="5.08" extent="1-16" drill="0.6"/>
+<contactref element="C1" pad="2"/>
 </signal>
 <signal name="N$20">
