File: v2/HWDesign/EAGLE/bluz_proto_v2_revA.sch (EAGLE design)
At the start: 69 parts

Commit message: add more breakouts. add decoupling cap
Parts:
- added C1: (no value), SparkFun-Capacitors:CAP0603-CAP
- added JP15, JP16: (no value), SparkFun-Connectors:M08NO_SILK
Connections:
- net GND: now also C1.2
- net VCC: now also C1.1
Changed lines of the file:
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@@
 <part name="S1" library="Spark" deviceset="TAC_SWITCH" device="SMD"/>
 <part name="GND5" library="SparkFun-Aesthetics" deviceset="GND" device=""/>
+<part name="C1" library="SparkFun-Capacitors" deviceset="CAP" device="0603-CAP"/>
+<part name="JP15" library="SparkFun-Connectors" deviceset="M08" device="NO_SILK"/>
+<part name="JP16" library="SparkFun-Connectors" deviceset="M08" device="NO_SILK"/>
 </parts>
 <sheets>
@@
 <instance part="JP9" gate="G$1" x="208.28" y="86.36"/>
 <instance part="JP10" gate="G$1" x="238.76" y="86.36"/>
-<instance part="GND2" gate="1" x="81.28" y="33.02"/>
-<instance part="SUPPLY2" gate="G$1" x="81.28" y="99.06"/>
+<instance part="GND2" gate="1" x="93.98" y="38.1"/>
+<instance part="SUPPLY2" gate="G$1" x="93.98" y="99.06"/>
 <instance part="JP11" gate="G$1" x="139.7" y="50.8"/>
 <instance part="JP12" gate="G$1" x="177.8" y="50.8"/>
@@
 <instance part="S1" gate="S" x="40.64" y="165.1"/>
 <instance part="GND5" gate="1" x="193.04" y="157.48"/>
+<instance part="C1" gate="G$1" x="93.98" y="88.9"/>
+<instance part="JP15" gate="G$1" x="264.16" y="86.36"/>
+<instance part="JP16" gate="G$1" x="264.16" y="50.8"/>
 </instances>
 <busses>
@@
 <junction x="73.66" y="91.44"/>
 <pinref part="SUPPLY2" gate="G$1" pin="VCC"/>
-<wire x1="73.66" y1="93.98" x2="81.28" y2="93.98" width="0.1524" layer="91"/>
-<wire x1="81.28" y1="93.98" x2="81.28" y2="99.06" width="0.1524" layer="91"/>
+<wire x1="73.66" y1="93.98" x2="93.98" y2="93.98" width="0.1524" layer="91"/>
+<wire x1="93.98" y1="93.98" x2="93.98" y2="99.06" width="0.1524" layer="91"/>
 <junction x="73.66" y="93.98"/>
+<pinref part="C1" gate="G$1" pin="1"/>
+<junction x="93.98" y="93.98"/>
 </segment>
 <segment>
@@
 <junction x="73.66" y="43.18"/>
 <pinref part="GND2" gate="1" pin="GND"/>
-<wire x1="73.66" y1="40.64" x2="81.28" y2="40.64" width="0.1524" layer="91"/>
-<wire x1="81.28" y1="40.64" x2="81.28" y2="35.56" width="0.1524" layer="91"/>
+<wire x1="73.66" y1="40.64" x2="93.98" y2="40.64" width="0.1524" layer="91"/>
 <junction x="73.66" y="40.64"/>
-</segment>
-<segment>
+<pinref part="C1" gate="G$1" pin="2"/>
+<wire x1="93.98" y1="86.36" x2="93.98" y2="40.64" width="0.1524" layer="91"/>
+<junction x="93.98" y="40.64"/>
+</segment>
+<segment>
